Commit message: Debug G1 + omnipicker assembly (#3)
* debug urdf

* single arm with gripper

* fixed dual arm + gripper debug urdf

* movable dual arm

* final G1 ver

File: manipulation/Agibot/agibot_g1_with_gripper_description/agibot_g1_with_omnipicker copy.urdf (robot description, URDF)
Before this commit: robot agibot_g1_with_omni-picker, 54 links, 53 joints
Links:
- link left_narrow2_Link: mass 0.0040132 -> 0.025428
- link right_narrow2_Link: mass 0.0040132 -> 0.025428
Joints:
- joint body_joint1: type prismatic -> fixed
- joint body_joint2: type revolute -> fixed
- joint head_joint1: type revolute -> fixed
- joint head_joint2: type revolute -> fixed
- joint left_camera_stand_base_joint: origin xyz=0.0 0.0 -0.0025 -> xyz=0.0 0.0 0.15
- joint left_camera_stand_mount_joint: origin xyz=0.0 0.0 0.005 -> xyz=0.0 0.0 0.3
- joint left_gripper_mount: origin xyz=0 0 0 rpy=0 0 1.57079632679 -> xyz=0 0 0.25 rpy=0 0 1.57079632679
- joint right_camera_stand_joint: origin xyz=0.0 0.0 -0.0025 -> xyz=0.0 0.0 0.15
- joint right_camera_stand_mount_joint: origin xyz=0.0 0.0 0.005 -> xyz=0.0 0.0 0.3
- joint right_gripper_mount: origin xyz=0 0 0 rpy=0 0 1.57079632679 -> xyz=0 0 0.25 rpy=0 0 1.57079632679

File: manipulation/Agibot/agibot_g1_with_gripper_description/agibot_g1_with_omnipicker.dual_fixed_arm.urdf (robot description, URDF)
Before this commit: robot agibot_g1_with_omni-picker, 54 links, 53 joints
Joints:
- joint body_joint1: type prismatic -> fixed
- joint body_joint2: type revolute -> fixed
- joint head_joint1: type revolute -> fixed
- joint head_joint2: type revolute -> fixed
- joint left_joint1: type revolute -> fixed
- joint left_joint2: type revolute -> fixed
- joint left_joint3: type revolute -> fixed
- joint left_joint4: type revolute -> fixed
- joint left_joint5: type revolute -> fixed
- joint left_joint6: type revolute -> fixed
- joint left_joint7: type revolute -> fixed
- joint right_joint1: type revolute -> fixed
- joint right_joint2: type revolute -> fixed
- joint right_joint3: type revolute -> fixed
- joint right_joint4: type revolute -> fixed
- joint right_joint5: type revolute -> fixed
- joint right_joint6: type revolute -> fixed
- joint right_joint7: type revolute -> fixed

File: manipulation/Agibot/agibot_g1_with_gripper_description/agibot_g1_with_omnipicker.dual_movable_arm.urdf (robot description, URDF)
Before this commit: robot agibot_g1_with_omni-picker, 54 links, 53 joints
Joints:
- joint body_joint1: type prismatic -> fixed
- joint body_joint2: type revolute -> fixed
- joint head_joint1: type revolute -> fixed
- joint head_joint2: type revolute -> fixed

File: manipulation/Agibot/agibot_g1_with_gripper_description/agibot_g1_with_omnipicker.single_fixed_arm.urdf (robot description, URDF)
Before this commit: robot agibot_g1_with_omni-picker, 54 links, 53 joints
Links:
- removed link arm_l_end_link
- removed link gripper_l_base_link
- removed link left_base_link
- removed link left_camera_stand
- removed link left_camera_stand_end
- removed link left_link1
- removed link left_link2
- removed link left_link3
- removed link left_link4
- removed link left_link5
- removed link left_link6
- removed link left_narrow1_Link
- removed link left_narrow2_Link
- removed link left_narrow3_Link
- removed link left_narrow4_Link
- removed link left_narrow_loop_Link
- removed link left_wide1_Link
- removed link left_wide2_Link
- removed link left_wide3_Link
- removed link left_wide4_Link
- removed link left_wide_loop_Link
- removed link right_narrow1_Link
- removed link right_narrow2_Link
- removed link right_narrow3_Link
- removed link right_narrow4_Link
- removed link right_narrow_loop_Link
- removed link right_wide1_Link
- removed link right_wide2_Link
- removed link right_wide3_Link
- removed link right_wide4_Link
- removed link right_wide_loop_Link
- added link narrow1_Link, mass 0.025428; collision mesh filename=meshes/omni_picker/narrow_1.obj; visual mesh filename=meshes/omni_picker/narrow_1.obj
- added link narrow2_Link, mass 0.0040132; collision mesh filename=meshes/omni_picker/narrow_2.obj; visual mesh filename=meshes/omni_picker/narrow_2.obj
- added link narrow3_Link, mass 0.018029; collision mesh filename=meshes/omni_picker/narrow_3.obj; visual mesh filename=meshes/omni_picker/narrow_3.obj
- added link narrow4_Link
- added link narrow_loop_Link, mass 0.022591; collision mesh filename=meshes/omni_picker/narrow_loop.obj; visual mesh filename=meshes/omni_picker/narrow_loop.obj
- added link wide1_Link, mass 0.025428; collision mesh filename=meshes/omni_picker/wide_1.obj; visual mesh filename=meshes/omni_picker/wide_1.obj
- added link wide2_Link, mass 0.0040132; collision mesh filename=meshes/omni_picker/wide_2.obj; visual mesh filename=meshes/omni_picker/wide_2.obj
- added link wide3_Link, mass 0.035835; collision mesh filename=meshes/omni_picker/wide_3.obj; visual mesh filename=meshes/omni_picker/wide_3.obj
- added link wide4_Link
- added link wide_loop_Link, mass 0.025142; collision mesh filename=meshes/omni_picker/wide_loop.obj; visual mesh filename=meshes/omni_picker/wide_loop.obj
Joints:
- removed joint left_base_joint
- removed joint left_camera_stand_base_joint
- removed joint left_camera_stand_mount_joint
- removed joint left_gripper_joint
- removed joint left_gripper_mount
- removed joint left_joint1
- removed joint left_joint2
- removed joint left_joint3
- removed joint left_joint4
- removed joint left_joint5
- removed joint left_joint6
- removed joint left_joint7
- removed joint left_narrow2_joint
- removed joint left_narrow3_joint
- removed joint left_narrow4_joint
- removed joint left_narrow_loop_joint
- removed joint left_wide1_joint
- removed joint left_wide2_joint
- removed joint left_wide3_joint
- removed joint left_wide4_joint
- removed joint left_wide_loop_joint
- removed joint right_gripper_joint
- removed joint right_narrow2_joint
- removed joint right_narrow3_joint
- removed joint right_narrow4_joint
- removed joint right_narrow_loop_joint
- removed joint right_wide1_joint
- removed joint right_wide2_joint
- removed joint right_wide3_joint
- removed joint right_wide4_joint
- removed joint right_wide_loop_joint
- added joint gripper_joint: type revolute, parent gripper_r_base_link, child narrow1_Link, origin xyz=0 -0.0195 0.0565 rpy=-2.9951 -1.5707963267948966 -0.15964, axis 0 0 1, limit lower=0 upper=1 effort=50 velocity=3.141592653589793
- added joint narrow2_joint: type revolute, parent narrow1_Link, child narrow2_Link, origin xyz=0.030852 0.018551 0, axis 0 0 -1, limit lower=-3.141592653589793 upper=3.141592653589793 effort=50 velocity=3.141592653589793, mimic joint=gripper_joint multiplier=0.02 offset=0
- added joint narrow3_joint: type revolute, parent narrow2_Link, child narrow3_Link, origin xyz=0.018118 -0.01574 0, axis 0 0 -1, limit lower=-3.141592653589793 upper=3.141592653589793 effort=50 velocity=3.141592653589793, mimic joint=gripper_joint multiplier=0.4 offset=0
- added joint narrow4_joint: type fixed, parent narrow3_Link, child narrow4_Link, origin xyz=0 -0.0104 0, axis 0 0 1, limit lower=-3.141592653589793 upper=3.141592653589793 effort=50 velocity=3.141592653589793
- added joint narrow_loop_joint: type revolute, parent gripper_r_base_link, child narrow_loop_Link, origin xyz=0 -0.021633 0.07387 rpy=-2.9951 -1.5707963267948966 -0.15964, axis 0 0 1, limit lower=-3.141592653589793 upper=3.141592653589793 effort=50 velocity=3.141592653589793, mimic joint=gripper_joint multiplier=1.5 offset=0
- added joint wide1_joint: type revolute, parent gripper_r_base_link, child wide1_Link, origin xyz=0 0.0195 0.0565 rpy=-2.9951 -1.5707963267948966 -0.15964, axis 0 0 -1, limit lower=-3.141592653589793 upper=3.141592653589793 effort=50 velocity=3.141592653589793, mimic joint=gripper_joint multiplier=1 offset=0
- added joint wide2_joint: type revolute, parent wide1_Link, child wide2_Link, origin xyz=0.030852 -0.018551 0, axis 0 0 1, limit lower=-3.141592653589793 upper=3.141592653589793 effort=50 velocity=3.141592653589793, mimic joint=gripper_joint multiplier=0.02 offset=0
- added joint wide3_joint: type revolute, parent wide2_Link, child wide3_Link, origin xyz=0.018118 0.01574 0, axis 0 0 1, limit lower=-3.141592653589793 upper=3.141592653589793 effort=50 velocity=3.141592653589793, mimic joint=gripper_joint multiplier=0.4 offset=0
- added joint wide4_joint: type fixed, parent wide3_Link, child wide4_Link, origin xyz=0 0.0104 0
- added joint wide_loop_joint: type revolute, parent gripper_r_base_link, child wide_loop_Link, origin xyz=0 0.021633 0.07387 rpy=-2.9951 -1.5707963267948966 -0.15964, axis 0 0 -1, limit lower=-3.141592653589793 upper=3.141592653589793 effort=50 velocity=3.141592653589793, mimic joint=gripper_joint multiplier=1.5 offset=0
- joint body_joint1: type prismatic -> fixed
- joint body_joint2: type revolute -> fixed
- joint head_joint1: type revolute -> fixed
- joint head_joint2: type revolute -> fixed
- joint right_joint1: type revolute -> fixed
- joint right_joint2: type revolute -> fixed
- joint right_joint3: type revolute -> fixed
- joint right_joint4: type revolute -> fixed
- joint right_joint5: type revolute -> fixed
- joint right_joint6: type revolute -> fixed
- joint right_joint7: type revolute -> fixed

File: manipulation/Agibot/agibot_g1_with_gripper_description/agibot_g1_with_omnipicker.single_movable_arm.urdf (robot description, URDF)
Before this commit: robot agibot_g1_with_omni-picker, 54 links, 53 joints
Links:
- removed link arm_l_end_link
- removed link gripper_l_base_link
- removed link left_base_link
- removed link left_camera_stand
- removed link left_camera_stand_end
- removed link left_link1
- removed link left_link2
- removed link left_link3
- removed link left_link4
- removed link left_link5
- removed link left_link6
- removed link left_narrow1_Link
- removed link left_narrow2_Link
- removed link left_narrow3_Link
- removed link left_narrow4_Link
- removed link left_narrow_loop_Link
- removed link left_wide1_Link
- removed link left_wide2_Link
- removed link left_wide3_Link
- removed link left_wide4_Link
- removed link left_wide_loop_Link
- removed link right_narrow1_Link
- removed link right_narrow2_Link
- removed link right_narrow3_Link
- removed link right_narrow4_Link
- removed link right_narrow_loop_Link
- removed link right_wide1_Link
- removed link right_wide2_Link
- removed link right_wide3_Link
- removed link right_wide4_Link
- removed link right_wide_loop_Link
- added link narrow1_Link, mass 0.025428; collision mesh filename=meshes/omni_picker/narrow_1.obj; visual mesh filename=meshes/omni_picker/narrow_1.obj
- added link narrow2_Link, mass 0.0040132; collision mesh filename=meshes/omni_picker/narrow_2.obj; visual mesh filename=meshes/omni_picker/narrow_2.obj
- added link narrow3_Link, mass 0.018029; collision mesh filename=meshes/omni_picker/narrow_3.obj; visual mesh filename=meshes/omni_picker/narrow_3.obj
- added link narrow4_Link
- added link narrow_loop_Link, mass 0.022591; collision mesh filename=meshes/omni_picker/narrow_loop.obj; visual mesh filename=meshes/omni_picker/narrow_loop.obj
- added link wide1_Link, mass 0.025428; collision mesh filename=meshes/omni_picker/wide_1.obj; visual mesh filename=meshes/omni_picker/wide_1.obj
- added link wide2_Link, mass 0.0040132; collision mesh filename=meshes/omni_picker/wide_2.obj; visual mesh filename=meshes/omni_picker/wide_2.obj
- added link wide3_Link, mass 0.035835; collision mesh filename=meshes/omni_picker/wide_3.obj; visual mesh filename=meshes/omni_picker/wide_3.obj
- added link wide4_Link
- added link wide_loop_Link, mass 0.025142; collision mesh filename=meshes/omni_picker/wide_loop.obj; visual mesh filename=meshes/omni_picker/wide_loop.obj
Joints:
- removed joint left_base_joint
- removed joint left_camera_stand_base_joint
- removed joint left_camera_stand_mount_joint
- removed joint left_gripper_joint
- removed joint left_gripper_mount
- removed joint left_joint1
- removed joint left_joint2
- removed joint left_joint3
- removed joint left_joint4
- removed joint left_joint5
- removed joint left_joint6
- removed joint left_joint7
- removed joint left_narrow2_joint
- removed joint left_narrow3_joint
- removed joint left_narrow4_joint
- removed joint left_narrow_loop_joint
- removed joint left_wide1_joint
- removed joint left_wide2_joint
- removed joint left_wide3_joint
- removed joint left_wide4_joint
- removed joint left_wide_loop_joint
- removed joint right_gripper_joint
- removed joint right_narrow2_joint
- removed joint right_narrow3_joint
- removed joint right_narrow4_joint
- removed joint right_narrow_loop_joint
- removed joint right_wide1_joint
- removed joint right_wide2_joint
- removed joint right_wide3_joint
- removed joint right_wide4_joint
- removed joint right_wide_loop_joint
- added joint gripper_joint: type revolute, parent gripper_r_base_link, child narrow1_Link, origin xyz=0 -0.0195 0.0565 rpy=-2.9951 -1.5707963267948966 -0.15964, axis 0 0 1, limit lower=0 upper=0.789 effort=50 velocity=3.141592653589793
- added joint narrow2_joint: type revolute, parent narrow1_Link, child narrow2_Link, origin xyz=0.030852 0.018551 0, axis 0 0 -1, limit lower=-3.141592653589793 upper=3.141592653589793 effort=50 velocity=3.141592653589793, mimic joint=gripper_joint multiplier=0.02 offset=0
- added joint narrow3_joint: type revolute, parent narrow2_Link, child narrow3_Link, origin xyz=0.018118 -0.01574 0, axis 0 0 -1, limit lower=-3.141592653589793 upper=3.141592653589793 effort=50 velocity=3.141592653589793, mimic joint=gripper_joint multiplier=0.4 offset=0
- added joint narrow4_joint: type fixed, parent narrow3_Link, child narrow4_Link, origin xyz=0 -0.0104 0, axis 0 0 1, limit lower=-3.141592653589793 upper=3.141592653589793 effort=50 velocity=3.141592653589793
- added joint narrow_loop_joint: type revolute, parent gripper_r_base_link, child narrow_loop_Link, origin xyz=0 -0.021633 0.07387 rpy=-2.9951 -1.5707963267948966 -0.15964, axis 0 0 1, limit lower=-3.141592653589793 upper=3.141592653589793 effort=50 velocity=3.141592653589793, mimic joint=gripper_joint multiplier=1.5 offset=0
- added joint wide1_joint: type revolute, parent gripper_r_base_link, child wide1_Link, origin xyz=0 0.0195 0.0565 rpy=-2.9951 -1.5707963267948966 -0.15964, axis 0 0 -1, limit lower=-3.141592653589793 upper=3.141592653589793 effort=50 velocity=3.141592653589793, mimic joint=gripper_joint multiplier=1 offset=0
- added joint wide2_joint: type revolute, parent wide1_Link, child wide2_Link, origin xyz=0.030852 -0.018551 0, axis 0 0 1, limit lower=-3.141592653589793 upper=3.141592653589793 effort=50 velocity=3.141592653589793, mimic joint=gripper_joint multiplier=0.02 offset=0
- added joint wide3_joint: type revolute, parent wide2_Link, child wide3_Link, origin xyz=0.018118 0.01574 0, axis 0 0 1, limit lower=-3.141592653589793 upper=3.141592653589793 effort=50 velocity=3.141592653589793, mimic joint=gripper_joint multiplier=0.4 offset=0
- added joint wide4_joint: type fixed, parent wide3_Link, child wide4_Link, origin xyz=0 0.0104 0
- added joint wide_loop_joint: type revolute, parent gripper_r_base_link, child wide_loop_Link, origin xyz=0 0.021633 0.07387 rpy=-2.9951 -1.5707963267948966 -0.15964, axis 0 0 -1, limit lower=-3.141592653589793 upper=3.141592653589793 effort=50 velocity=3.141592653589793, mimic joint=gripper_joint multiplier=1.5 offset=0
- joint body_joint1: type prismatic -> fixed
- joint body_joint2: type revolute -> fixed
- joint head_joint1: type revolute -> fixed
- joint head_joint2: type revolute -> fixed

File: manipulation/Agibot/agibot_g1_with_gripper_description/agibot_g1_with_omnipicker_gripperbase.urdf (robot description, URDF)
Before this commit: robot agibot_g1_with_omni-picker, 54 links, 53 joints
Links:
- removed link left_narrow1_Link
- removed link left_narrow2_Link
- removed link left_narrow3_Link
- removed link left_narrow4_Link
- removed link left_narrow_loop_Link
- removed link left_wide1_Link
- removed link left_wide2_Link
- removed link left_wide3_Link
- removed link left_wide4_Link
- removed link left_wide_loop_Link
- removed link right_narrow1_Link
- removed link right_narrow2_Link
- removed link right_narrow3_Link
- removed link right_narrow4_Link
- removed link right_narrow_loop_Link
- removed link right_wide1_Link
- removed link right_wide2_Link
- removed link right_wide3_Link
- removed link right_wide4_Link
- removed link right_wide_loop_Link
Joints:
- removed joint left_gripper_joint
- removed joint left_narrow2_joint
- removed joint left_narrow3_joint
- removed joint left_narrow4_joint
- removed joint left_narrow_loop_joint
- removed joint left_wide1_joint
- removed joint left_wide2_joint
- removed joint left_wide3_joint
- removed joint left_wide4_joint
- removed joint left_wide_loop_joint
- removed joint right_gripper_joint
- removed joint right_narrow2_joint
- removed joint right_narrow3_joint
- removed joint right_narrow4_joint
- removed joint right_narrow_loop_joint
- removed joint right_wide1_joint
- removed joint right_wide2_joint
- removed joint right_wide3_joint
- removed joint right_wide4_joint
- removed joint right_wide_loop_joint
- joint body_joint1: type prismatic -> fixed
- joint body_joint2: type revolute -> fixed
- joint head_joint1: type revolute -> fixed
- joint head_joint2: type revolute -> fixed
