Commit message: a worked without camera stand

File: manipulation/Agibot/agibot_g1_with_gripper_description/agibot_g1_with_omnipicker.urdf (robot description, URDF)
Before this commit: robot agibot_g1_with_omni-picker, 52 links, 51 joints
Links:
- removed link left_eef
- removed link left_end_link
- removed link left_gripper_base
- removed link right_eef
- removed link right_gripper_base
- added link arm_l_end_link, mass 0.06158; collision cylinder length=0.045999998692423105 radius=0.030799950382754494; visual mesh filename=meshes/arm/link7.obj
- added link gripper_l_base_link, mass 0.25641368; visual mesh filename=meshes/omni_picker/gripper_base.obj
- added link gripper_r_base_link, mass 0.25641368; visual mesh filename=meshes/omni_picker/gripper_base.obj
- added link left_camera_stand
- added link right_camera_stand
Joints:
- removed joint left_eef_joint
- removed joint right_eef_joint
- added joint left_camera_stand_joint: type fixed, parent arm_l_end_link, child left_camera_stand, origin xyz=0.0 0.0 0.005
- added joint right_camera_stand_joint: type fixed, parent right_end_link, child right_camera_stand, origin xyz=0.0 0.0 0.005
- joint left_gripper_joint: parent left_gripper_base -> gripper_l_base_link
- joint left_gripper_mount: child left_gripper_base -> gripper_l_base_link; origin xyz=0 0 0 rpy=0 0 0 -> rpy=0 0 1.57079632679; parent left_eef -> left_camera_stand
- joint left_joint7: child left_end_link -> arm_l_end_link
- joint left_narrow_loop_joint: parent left_gripper_base -> gripper_l_base_link
- joint left_wide1_joint: parent left_gripper_base -> gripper_l_base_link
- joint left_wide_loop_joint: parent left_gripper_base -> gripper_l_base_link
- joint right_gripper_joint: parent right_gripper_base -> gripper_r_base_link
- joint right_gripper_mount: child right_gripper_base -> gripper_r_base_link; origin xyz=0 0 0 rpy=0 0 0 -> xyz=0 0 0 rpy=0 0 1.57079632679; parent right_eef -> right_camera_stand
- joint right_narrow_loop_joint: parent right_gripper_base -> gripper_r_base_link
- joint right_wide1_joint: parent right_gripper_base -> gripper_r_base_link
- joint right_wide_loop_joint: parent right_gripper_base -> gripper_r_base_link

Commit message: mount left camera stand

File: manipulation/Agibot/agibot_g1_with_gripper_description/agibot_g1_with_omnipicker.urdf (robot description, URDF)
Before this commit: robot agibot_g1_with_omni-picker, 52 links, 51 joints
Links:
- added link left_camera_stand_end
- link left_camera_stand: geometry visual mesh filename=meshes/camera/120s_camera_stand.obj
Joints:
- removed joint left_camera_stand_joint
- added joint left_camera_stand_base_joint: type fixed, parent arm_l_end_link, child left_camera_stand, origin xyz=0.0 0.0 0.0
- added joint left_camera_stand_mount_joint: type fixed, parent left_camera_stand, child left_camera_stand_end, origin xyz=0.0 0.0 0.005

Commit message: mount stand fix

File: manipulation/Agibot/agibot_g1_with_gripper_description/agibot_g1_with_omnipicker.urdf (robot description, URDF)
Before this commit: robot agibot_g1_with_omni-picker, 53 links, 52 joints
Links:
- removed link right_end_link
- added link arm_r_end_link, mass 0.06158; collision cylinder length=0.045999998692423105 radius=0.030799950382754494; visual mesh filename=meshes/arm/link7.obj
- added link right_camera_stand_end
- link right_camera_stand: geometry visual mesh filename=meshes/camera/120s_camera_stand.obj
Joints:
- added joint right_camera_stand_mount_joint: type fixed, parent right_camera_stand, child right_camera_stand_end, origin xyz=0.0 0.0 0.005
- joint left_gripper_mount: origin rpy=0 0 1.57079632679 -> xyz=0 0 0 rpy=0 0 1.57079632679; parent left_camera_stand -> left_camera_stand_end
- joint right_camera_stand_joint: origin xyz=0.0 0.0 0.005 -> xyz=0.0 0.0 0.0; parent right_end_link -> arm_r_end_link
- joint right_gripper_mount: parent right_camera_stand -> right_camera_stand_end
- joint right_joint7: child right_end_link -> arm_r_end_link

Commit message: fixed flange pose

File: manipulation/Agibot/agibot_g1_with_gripper_description/agibot_g1_with_omnipicker.urdf (robot description, URDF)
Before this commit: robot agibot_g1_with_omni-picker, 54 links, 53 joints
Links:
- link left_camera_stand: geometry visual mesh filename=meshes/camera/omni_picker_camera_stand.obj
- link right_camera_stand: geometry visual mesh filename=meshes/camera/omni_picker_camera_stand.obj
Joints:
- joint left_camera_stand_base_joint: origin xyz=0.0 0.0 0.0 -> xyz=0.0 0.0 -0.0025
- joint right_camera_stand_joint: origin xyz=0.0 0.0 0.0 -> xyz=0.0 0.0 -0.0025

Commit message: G1_omnipicker URDF assemble (#1)
* mesh use relative path

* a worked without camera stand

* mount left camera stand

* mount stand fix

* fixed flange pose

* done g1_omnipicker with readme

File: manipulation/Agibot/agibot_g1_with_gripper_description/agibot_g1_with_omnipicker.urdf (robot description, URDF)
Before this commit: robot agibot_g1_with_omni-picker, 52 links, 51 joints
Links:
- removed link left_eef
- removed link left_end_link
- removed link left_gripper_base
- removed link right_eef
- removed link right_end_link
- removed link right_gripper_base
- added link arm_l_end_link, mass 0.06158; collision cylinder length=0.045999998692423105 radius=0.030799950382754494; visual mesh filename=meshes/arm/link7.obj
- added link arm_r_end_link, mass 0.06158; collision cylinder length=0.045999998692423105 radius=0.030799950382754494; visual mesh filename=meshes/arm/link7.obj
- added link gripper_l_base_link, mass 0.25641368; visual mesh filename=meshes/omni_picker/gripper_base.obj
- added link gripper_r_base_link, mass 0.25641368; visual mesh filename=meshes/omni_picker/gripper_base.obj
- added link left_camera_stand; visual mesh filename=meshes/camera/omni_picker_camera_stand.obj
- added link left_camera_stand_end
- added link right_camera_stand; visual mesh filename=meshes/camera/omni_picker_camera_stand.obj
- added link right_camera_stand_end
- link base_link: geometry collision box size=0.29833984 0.3376392 1.0; collision box size=0.5796094 0.449 0.27073438
- link body_link1: geometry collision box size=0.16064453 0.05555534399999999 0.1328125; collision box size=0.16259765999999998 0.04375648500000001 0.16015625
- link body_link2: geometry collision box size=0.34570312 0.18107724 0.3125; collision cylinder length=0.08697056999999997 radius=0.09662318
- link head_link1: geometry visual mesh filename=meshes/base/head_link1.obj
- link head_link2: geometry collision sphere radius=0.11257068650657154; visual mesh filename=meshes/base/head_link2.obj
- link left_base_link: geometry visual mesh filename=meshes/arm/base_link.obj
- link left_link1: geometry collision cylinder length=0.16642063483595848 radius=0.05579268228774888; visual mesh filename=meshes/arm/link1.obj
- link left_link2: geometry collision cylinder length=0.18085919 radius=0.06302423; visual mesh filename=meshes/arm/link2.obj
- link left_link3: geometry collision cylinder length=0.22061403840780258 radius=0.05216156143823925; visual mesh filename=meshes/arm/link3.obj
- link left_link4: geometry collision cylinder length=0.154955404 radius=0.057891708; visual mesh filename=meshes/arm/link4.obj
- link left_link5: geometry collision cylinder length=0.13423806056380272 radius=0.04562028545392604; visual mesh filename=meshes/arm/link5.obj
- link left_link6: geometry collision cylinder length=0.18272488500982115 radius=0.04857149291994264; visual mesh filename=meshes/arm/link6.obj
- link left_narrow1_Link: geometry collision mesh filename=meshes/omni_picker/narrow_1.obj; visual mesh filename=meshes/omni_picker/narrow_1.obj
- link left_narrow2_Link: geometry collision mesh filename=meshes/omni_picker/narrow_2.obj; visual mesh filename=meshes/omni_picker/narrow_2.obj
- link left_narrow3_Link: geometry collision mesh filename=meshes/omni_picker/narrow_3.obj; visual mesh filename=meshes/omni_picker/narrow_3.obj
- link left_narrow_loop_Link: geometry collision mesh filename=meshes/omni_picker/narrow_loop.obj; visual mesh filename=meshes/omni_picker/narrow_loop.obj
- link left_wide1_Link: geometry collision mesh filename=meshes/omni_picker/wide_1.obj; visual mesh filename=meshes/omni_picker/wide_1.obj
- link left_wide2_Link: geometry collision mesh filename=meshes/omni_picker/wide_2.obj; visual mesh filename=meshes/omni_picker/wide_2.obj
- link left_wide3_Link: geometry collision mesh filename=meshes/omni_picker/wide_3.obj; visual mesh filename=meshes/omni_picker/wide_3.obj
- link left_wide_loop_Link: geometry collision mesh filename=meshes/omni_picker/wide_loop.obj; visual mesh filename=meshes/omni_picker/wide_loop.obj
- link right_base_link: geometry visual mesh filename=meshes/arm/base_link.obj
- link right_link1: geometry collision cylinder length=0.16642063483595848 radius=0.05579268228774888; visual mesh filename=meshes/arm/link1.obj
- link right_link2: geometry collision cylinder length=0.18085919 radius=0.06302423; visual mesh filename=meshes/arm/link2.obj
- link right_link3: geometry collision cylinder length=0.22061403840780258 radius=0.05216156143823925; visual mesh filename=meshes/arm/link3.obj
- link right_link4: geometry collision cylinder length=0.154955404 radius=0.057891708; visual mesh filename=meshes/arm/link4.obj
- link right_link5: geometry collision cylinder length=0.13423806056380272 radius=0.04562028545392604; visual mesh filename=meshes/arm/link5.obj
- link right_link6: geometry collision cylinder length=0.18272488500982115 radius=0.04857149291994264; visual mesh filename=meshes/arm/link6.obj
- link right_narrow1_Link: geometry collision mesh filename=meshes/omni_picker/narrow_1.obj; visual mesh filename=meshes/omni_picker/narrow_1.obj
- link right_narrow2_Link: geometry collision mesh filename=meshes/omni_picker/narrow_2.obj; visual mesh filename=meshes/omni_picker/narrow_2.obj
- link right_narrow3_Link: geometry collision mesh filename=meshes/omni_picker/narrow_3.obj; visual mesh filename=meshes/omni_picker/narrow_3.obj
- link right_narrow_loop_Link: geometry collision mesh filename=meshes/omni_picker/narrow_loop.obj; visual mesh filename=meshes/omni_picker/narrow_loop.obj
- link right_wide1_Link: geometry collision mesh filename=meshes/omni_picker/wide_1.obj; visual mesh filename=meshes/omni_picker/wide_1.obj
- link right_wide2_Link: geometry collision mesh filename=meshes/omni_picker/wide_2.obj; visual mesh filename=meshes/omni_picker/wide_2.obj
- link right_wide3_Link: geometry collision mesh filename=meshes/omni_picker/wide_3.obj; visual mesh filename=meshes/omni_picker/wide_3.obj
- link right_wide_loop_Link: geometry collision mesh filename=meshes/omni_picker/wide_loop.obj; visual mesh filename=meshes/omni_picker/wide_loop.obj
Joints:
- removed joint left_eef_joint
- removed joint right_eef_joint
- added joint left_camera_stand_base_joint: type fixed, parent arm_l_end_link, child left_camera_stand, origin xyz=0.0 0.0 -0.0025
- added joint left_camera_stand_mount_joint: type fixed, parent left_camera_stand, child left_camera_stand_end, origin xyz=0.0 0.0 0.005
- added joint right_camera_stand_joint: type fixed, parent arm_r_end_link, child right_camera_stand, origin xyz=0.0 0.0 -0.0025
- added joint right_camera_stand_mount_joint: type fixed, parent right_camera_stand, child right_camera_stand_end, origin xyz=0.0 0.0 0.005
- joint left_gripper_joint: parent left_gripper_base -> gripper_l_base_link
- joint left_gripper_mount: child left_gripper_base -> gripper_l_base_link; origin xyz=0 0 0 rpy=0 0 0 -> xyz=0 0 0 rpy=0 0 1.57079632679; parent left_eef -> left_camera_stand_end
- joint left_joint7: child left_end_link -> arm_l_end_link
- joint left_narrow_loop_joint: parent left_gripper_base -> gripper_l_base_link
- joint left_wide1_joint: parent left_gripper_base -> gripper_l_base_link
- joint left_wide_loop_joint: parent left_gripper_base -> gripper_l_base_link
- joint right_gripper_joint: parent right_gripper_base -> gripper_r_base_link
- joint right_gripper_mount: child right_gripper_base -> gripper_r_base_link; origin xyz=0 0 0 rpy=0 0 0 -> xyz=0 0 0 rpy=0 0 1.57079632679; parent right_eef -> right_camera_stand_end
- joint right_joint7: child right_end_link -> arm_r_end_link
- joint right_narrow_loop_joint: parent right_gripper_base -> gripper_r_base_link
- joint right_wide1_joint: parent right_gripper_base -> gripper_r_base_link
- joint right_wide_loop_joint: parent right_gripper_base -> gripper_r_base_link

Commit message: final G1 ver

File: manipulation/Agibot/agibot_g1_with_gripper_description/agibot_g1_with_omnipicker.urdf (robot description, URDF)
Before this commit: robot agibot_g1_with_omni-picker, 54 links, 53 joints
Joints:
- joint body_joint1: type fixed -> prismatic
- joint body_joint2: type fixed -> revolute
- joint head_joint1: type fixed -> revolute
- joint head_joint2: type fixed -> revolute
- joint left_gripper_mount: origin xyz=0 0 0.2 rpy=0 0 1.57079632679 -> xyz=0 0 0 rpy=0 0 1.57079632679
- joint left_joint1: type fixed -> revolute
- joint left_joint2: type fixed -> revolute
- joint left_joint3: type fixed -> revolute
- joint left_joint4: type fixed -> revolute
- joint left_joint5: type fixed -> revolute
- joint left_joint6: type fixed -> revolute
- joint left_joint7: type fixed -> revolute
- joint right_gripper_mount: origin xyz=0 0 0.2 rpy=0 0 1.57079632679 -> xyz=0 0 0 rpy=0 0 1.57079632679
- joint right_joint1: type fixed -> revolute
- joint right_joint2: type fixed -> revolute
- joint right_joint3: type fixed -> revolute
- joint right_joint4: type fixed -> revolute
- joint right_joint5: type fixed -> revolute
- joint right_joint6: type fixed -> revolute
- joint right_joint7: type fixed -> revolute

Commit message: limit gripper joint

File: manipulation/Agibot/agibot_g1_with_gripper_description/agibot_g1_with_omnipicker.urdf (robot description, URDF)
Before this commit: robot agibot_g1_with_omni-picker, 54 links, 53 joints
Joints:
- joint left_gripper_joint: limit lower=0 upper=1 effort=50 velocity=3.141592653589793 -> lower=0.1 upper=0.78 effort=50 velocity=3.141592653589793
- joint right_gripper_joint: limit lower=0 upper=1 effort=50 velocity=3.141592653589793 -> lower=0.1 upper=0.785 effort=50 velocity=3.141592653589793

Commit message: fix right gripper mount ori

File: manipulation/Agibot/agibot_g1_with_gripper_description/agibot_g1_with_omnipicker.urdf (robot description, URDF)
Before this commit: robot agibot_g1_with_omni-picker, 54 links, 53 joints
Joints:
- joint right_gripper_mount: origin xyz=0 0 0 rpy=0 0 1.57079632679 -> xyz=0 0 0 rpy=0 0 -1.57079632679
