Commit message: fixed wheel

File: manipulation/Agibot/agibot_g1_description/urdf/agibot_g1_omni-picker.urdf (robot description, URDF)
Before this commit: robot Agibot G1, 30 links, 29 joints
Links:
- link base_link: geometry collision box size=0.29833984 0.3376392 1.0; collision box size=0.5796094 0.449 0.27073438
- link body_link1: geometry collision box size=0.16064453 0.05555534399999999 0.1328125; collision box size=0.16259765999999998 0.04375648500000001 0.16015625
- link body_link2: geometry collision box size=0.34570312 0.18107724 0.3125; collision cylinder length=0.08697056999999997 radius=0.09662318
- link head_link1: geometry visual mesh filename=../meshes/base/head_link1.obj
- link head_link2: geometry collision sphere radius=0.11257068650657154; visual mesh filename=../meshes/base/head_link2.obj
- link left_base_link: geometry visual mesh filename=../meshes/arm/base_link.obj
- link left_end_link: geometry collision cylinder length=0.045999998692423105 radius=0.030799950382754494; visual mesh filename=../meshes/arm/link7.obj
- link left_link1: geometry collision cylinder length=0.16642063483595848 radius=0.05579268228774888; visual mesh filename=../meshes/arm/link1.obj
- link left_link2: geometry collision cylinder length=0.18085919 radius=0.06302423; visual mesh filename=../meshes/arm/link2.obj
- link left_link3: geometry collision cylinder length=0.22061403840780258 radius=0.05216156143823925; visual mesh filename=../meshes/arm/link3.obj
- link left_link4: geometry collision cylinder length=0.154955404 radius=0.057891708; visual mesh filename=../meshes/arm/link4.obj
- link left_link5: geometry collision cylinder length=0.13423806056380272 radius=0.04562028545392604; visual mesh filename=../meshes/arm/link5.obj
- link left_link6: geometry collision cylinder length=0.18272488500982115 radius=0.04857149291994264; visual mesh filename=../meshes/arm/link6.obj
- link right_base_link: geometry visual mesh filename=../meshes/arm/base_link.obj
- link right_end_link: geometry collision cylinder length=0.045999998692423105 radius=0.030799950382754494; visual mesh filename=../meshes/arm/link7.obj
- link right_link1: geometry collision cylinder length=0.16642063483595848 radius=0.05579268228774888; visual mesh filename=../meshes/arm/link1.obj
- link right_link2: geometry collision cylinder length=0.18085919 radius=0.06302423; visual mesh filename=../meshes/arm/link2.obj
- link right_link3: geometry collision cylinder length=0.22061403840780258 radius=0.05216156143823925; visual mesh filename=../meshes/arm/link3.obj
- link right_link4: geometry collision cylinder length=0.154955404 radius=0.057891708; visual mesh filename=../meshes/arm/link4.obj
- link right_link5: geometry collision cylinder length=0.13423806056380272 radius=0.04562028545392604; visual mesh filename=../meshes/arm/link5.obj
- link right_link6: geometry collision cylinder length=0.18272488500982115 radius=0.04857149291994264; visual mesh filename=../meshes/arm/link6.obj
Joints:
- joint left_wheel_joint: type continuous -> fixed
- joint right_wheel_joint: type continuous -> fixed

File: manipulation/Agibot/agibot_g1_with_gripper_description/agibot_g1_with_omnipicker.urdf (robot description, URDF)
Before this commit: robot agibot_g1_with_omni-picker, 54 links, 53 joints
Joints:
- joint left_wheel_joint: type continuous -> fixed
- joint right_wheel_joint: type continuous -> fixed

Commit message: consistent with urdf in geniesim assets

File: manipulation/Agibot/agibot_g1_description/urdf/agibot_g1_omni-picker.urdf (robot description, URDF)
Before this commit: robot Agibot G1, 30 links, 29 joints
Joints:
- joint right_joint1: axis 0.0 0.0 -1.0 -> 0.0 0.0 1.0
- joint right_joint2: axis 0.0 0.0 -1.0 -> 0.0 0.0 1.0
- joint right_joint3: axis 0.0 0.0 -1.0 -> 0.0 0.0 1.0
- joint right_joint4: axis 0.0 0.0 -1.0 -> 0.0 0.0 1.0
- joint right_joint5: axis 0.0 0.0 -1.0 -> 0.0 0.0 1.0
- joint right_joint6: axis 0.0 0.0 -1.0 -> 0.0 0.0 1.0
- joint right_joint7: axis 0.0 0.0 -1.0 -> 0.0 0.0 1.0
